Commit message: update

File: description/face.xacro (robot description, xacro)
@@ -4,5 +4,5 @@
         <parent link="chassis"/>
         <child link="face_link"/>
-        <origin xyz="${chassis_length} 0 ${chassis_height/2}" rpy="0 0 0"/>
+        <origin xyz="${chassis_length}/2 0 ${chassis_height/2}" rpy="0 0 0"/>
     </joint>
     <link name="face_link">

File: description/robot_core.xacro (robot description, xacro)
@@ -164,5 +164,5 @@
         <parent link="chassis"/>
         <child link="laser_frame"/>
-        <origin xyz="${chassis_length -0.150} 0 ${chassis_height + 0.030}" rpy="0 0 0"/>
+        <origin xyz="${chassis_length/2 -0.150} 0 ${chassis_height + 0.030}" rpy="0 0 0"/>
     </joint>
     <link name="laser_frame">

Commit message: update

File: description/face.xacro (robot description, xacro)
@@ -4,5 +4,5 @@
         <parent link="chassis"/>
         <child link="face_link"/>
-        <origin xyz="${chassis_length}/2 0 ${chassis_height/2}" rpy="0 0 0"/>
+        <origin xyz="${chassis_length/2} 0 ${chassis_height/2}" rpy="0 0 0"/>
     </joint>
     <link name="face_link">

File: description/robot_core.xacro (robot description, xacro)
@@ -58,5 +58,5 @@
         <parent link="base_link"/>
         <child link="chassis"/>
-        <origin xyz="0 0 ${-wheel_offset_z}"/>
+        <origin xyz="-${chassis_length/2} 0 ${-wheel_offset_z}"/>
     </joint>
     <link name="chassis">
@@ -83,5 +83,5 @@
     <!-- LEFT WHEEL LINK -->
     <joint name="left_wheel_joint" type="continuous">
-        <parent link="base_link"/>
+        <parent link="chassis"/>
         <child link="left_wheel"/>
         <origin xyz="${chassis_length/2 - 0.070} ${wheel_offset_y/2 + wheel_thickness/2 + 0.01} 0" rpy="-${pi/2} 0 0" />
@@ -109,5 +109,5 @@
     <!-- RIGHT WHEEL LINK -->
     <joint name="right_wheel_joint" type="continuous">
-        <parent link="base_link"/>
+        <parent link="chassis"/>
         <child link="right_wheel"/>
         <origin xyz="${chassis_length/2 - 0.070} -${wheel_offset_y/2 + wheel_thickness/2 + 0.01} 0" rpy="${pi/2} 0 0" />
@@ -137,5 +137,5 @@
         <parent link="chassis"/>
         <child link="caster_wheel"/>
-        <origin xyz="${caster_wheel_offset_x} 0 ${caster_wheel_offset_z}"/>
+        <origin xyz="-${caster_wheel_offset_x*2} 0 ${caster_wheel_offset_z}"/>
     </joint>
     <link name="caster_wheel">
