Commit message: update

File: description/imu.xacro (robot description, xacro)
@@ -4,5 +4,5 @@
         <parent link="chassis"/>
         <child link="imu_link"/>
-        <origin xyz="${chassis_length/2 - 0.15285} 0 ${chassis_height/2}" rpy="0 0 0"/>
+        <origin xyz="${chassis_length/2 - 0.15285} 0 0}" rpy="0 0 0"/>
     </joint>
     <link name="imu_link">

Commit message: update

File: description/imu.xacro (robot description, xacro)
@@ -4,5 +4,5 @@
         <parent link="chassis"/>
         <child link="imu_link"/>
-        <origin xyz="${chassis_length/2 - 0.15285} 0 0}" rpy="0 0 0"/>
+        <origin xyz="${chassis_length/2 - 0.15285} 0 ${chassis_height/2}" rpy="0 0 0"/>
     </joint>
     <link name="imu_link">

Commit message: update

File: description/imu.xacro (robot description, xacro)
@@ -4,5 +4,5 @@
         <parent link="chassis"/>
         <child link="imu_link"/>
-        <origin xyz="${chassis_length/2 - 0.15285} 0 ${chassis_height/2}" rpy="0 0 0"/>
+        <origin xyz="${chassis_length/2 - 0.15285} 0 0" rpy="0 0 0"/>
     </joint>
     <link name="imu_link">

Commit message: update

File: description/imu.xacro (robot description, xacro)
@@ -6,7 +6,7 @@
         <origin xyz="${chassis_length/2 - 0.15285} 0 0" rpy="0 0 0"/>
     </joint>
-    <link name="imu_link">
+    <link name="imu">
     </link>
-    <gazebo reference="imu_link">
+    <gazebo reference="imu">
         <material>Gazebo/Black</material>
     </gazebo>

File: description/robot_core.xacro (robot description, xacro)
@@ -206,24 +206,3 @@
         <material>Gazebo/White</material>
     </gazebo>
-    <joint name="imu_joint" type="fixed">
-        <parent link="chassis"/>
-        <child link="imu"/>
-        <origin xyz="${chassis_length/2 - 0.15285} 0 ${chassis_height/2 + 0.030}" rpy="0 0 ${pi}"/>
-    </joint>
-    <link name="imu">
-        <visual>
-            <geometry>
-                <cylinder radius="0.04" length="0.05"/>
-            </geometry>
-            <material name="black"/>
-        </visual>
-        <collision>
-            <geometry>
-                <sphere radius="${caster_wheel_radius}"/>
-            </geometry>
-        </collision>
-        <xacro:inertial_sphere mass="${caster_wheel_mass}" radius="${caster_wheel_radius}">
-            <origin xyz="0 0 0" rpy="0 0 0"/>
-        </xacro:inertial_sphere>
-    </link>
 </robot>

Commit message: update

File: description/imu.xacro (robot description, xacro)
@@ -3,5 +3,5 @@
     <joint name="imu_joint" type="fixed">
         <parent link="chassis"/>
-        <child link="imu_link"/>
+        <child link="imu"/>
         <origin xyz="${chassis_length/2 - 0.15285} 0 0" rpy="0 0 0"/>
     </joint>

Commit message: update

File: description/imu.xacro (robot description, xacro)
@@ -3,10 +3,10 @@
     <joint name="imu_joint" type="fixed">
         <parent link="chassis"/>
-        <child link="imu"/>
+        <child link="robot_imu"/>
         <origin xyz="${chassis_length/2 - 0.15285} 0 0" rpy="0 0 0"/>
     </joint>
-    <link name="imu">
+    <link name="robot_imu">
     </link>
-    <gazebo reference="imu">
+    <gazebo reference="robot_imu">
         <material>Gazebo/Black</material>
     </gazebo>
