Commit message: update

File: description/camera.xacro (robot description, xacro)
@@ -4,5 +4,5 @@
         <parent link="chassis"/>
         <child link="camera_link"/>
-        <origin xyz="0.276 0 0.181" rpy="0 0 0"/>
+        <origin xyz="${chassis_length/2} 0 ${chassis_height/2}" rpy="0 0 0"/>
     </joint>
     <link name="camera_link">

Commit message: update

File: description/camera.xacro (robot description, xacro)
@@ -20,4 +20,12 @@
             <material name="black"/>
         </visual>
+    </link>
+    <!-- add camera_frame for realsense 21.01.2025 -->
+    <joint name="camera_frame_joint" type="fixed">
+        <parent link="chassis"/>
+        <child link="camera_frame"/>
+        <origin xyz="${chassis_length/2} 0 ${chassis_height/2 + 0.06}" rpy="0 0 0"/>
+    </joint>
+    <link name="camera_frame">
     </link>
     <joint name="camera_optical_joint" type="fixed">
