Commit message: update include femto mega

File: description/robot.urdf.xacro (robot description, xacro)
@@ -10,10 +10,8 @@
         <xacro:include filename="gazebo_control.xacro" />
     </xacro:unless>
-    <!-- <xacro:include filename="lidar.xacro" /> -->
-    <!-- <xacro:include filename="camera.xacro" /> -->
-    <!-- <xacro:include filename="depth_camera.xacro" /> -->
-    <!-- <xacro:include filename="face.xacro" /> -->
     <xacro:include filename="imu.xacro" />
-    <!-- New xacro file defining oak-d-lite depth camera -->
-    <xacro:include filename="oak-d-lite.xacro"/>
+    <!-- New xacro file defining oak-d-lite depth camera
+    <xacro:include filename="oak-d-lite.xacro"/> -->
+    <!-- femto_bolt xacro file -->
+    <xacro:include filename="femto_mega.urdf.xacro" />
 </robot>

File: description/robot_core.xacro (robot description, xacro)
@@ -160,26 +160,4 @@
         <mu2 value="0.001"/>
     </gazebo>
-    <!-- Lidar LINK -->
-    <!-- <joint name="lidar_joint" type="fixed">
-        <parent link="chassis"/>
-        <child link="laser_frame"/>
-        <origin xyz="${chassis_length/2 -0.150} 0 ${chassis_height + 0.030}" rpy="0 0 0"/>
-    </joint>
-    <link name="laser_frame">
-        <visual>
-            <geometry>
-                <sphere radius="${caster_wheel_radius}"/>
-            </geometry>
-            <material name="white"/>
-        </visual>
-        <collision>
-            <geometry>
-                <sphere radius="${caster_wheel_radius}"/>
-            </geometry>
-        </collision>
-        <xacro:inertial_sphere mass="${caster_wheel_mass}" radius="${caster_wheel_radius}">
-            <origin xyz="0 0 0" rpy="0 0 0"/>
-        </xacro:inertial_sphere>
-    </link> -->
     <joint name="laser_joint" type="fixed">
         <parent link="chassis"/>
