Commit message: update

File: description/femto_mega.urdf.xacro (robot description, xacro)
@@ -11,5 +11,6 @@
   <xacro:property name="cam_height" value="0.06495"/>
   <xacro:property name="cam_depth" value="0.04026"/>
-  <xacro:property name="mesh_path" value="models/" />
+  <!-- <xacro:property name="mesh_path" value="models/" /> -->
+  <xacro:property name="mesh_path" value="file://$(find my_package)/meshes/rp_lidar.dae" />
   <!-- The following values are approximate but the camera node
      publishes TF values with actual calibrated camera extrinsic values -->

Commit message: update package

File: description/femto_mega.urdf.xacro (robot description, xacro)
@@ -12,5 +12,5 @@
   <xacro:property name="cam_depth" value="0.04026"/>
   <!-- <xacro:property name="mesh_path" value="models/" /> -->
-  <xacro:property name="mesh_path" value="file://$(find my_package)/meshes/rp_lidar.dae" />
+  <xacro:property name="mesh_path" value="file://$(ros2_rmp_support)/description/models/" />
   <!-- The following values are approximate but the camera node
      publishes TF values with actual calibrated camera extrinsic values -->

Commit message: update

File: description/femto_mega.urdf.xacro (robot description, xacro)
@@ -12,5 +12,5 @@
   <xacro:property name="cam_depth" value="0.04026"/>
   <!-- <xacro:property name="mesh_path" value="models/" /> -->
-  <xacro:property name="mesh_path" value="file://$(ros2_rmp_support)/description/models/" />
+  <xacro:property name="mesh_path" value="models/" />
   <!-- The following values are approximate but the camera node
      publishes TF values with actual calibrated camera extrinsic values -->
