Commit message: update

File: description/robot_core.xacro (robot description, xacro)
@@ -160,3 +160,30 @@
         <mu2 value="0.001"/>
     </gazebo>
+    <!-- Lidar LINK -->
+    <joint name="lidar_joint" type="fixed">
+        <parent link="chassis"/>
+        <child link="laser_frame"/>
+        <origin xyz="-150 0 30"/>
+    </joint>
+    <link name="caster_wheel">
+        <visual>
+            <geometry>
+                <sphere radius="${caster_wheel_radius}"/>
+            </geometry>
+            <material name="white"/>
+        </visual>
+        <collision>
+            <geometry>
+                <sphere radius="${caster_wheel_radius}"/>
+            </geometry>
+        </collision>
+        <xacro:inertial_sphere mass="${caster_wheel_mass}" radius="${caster_wheel_radius}">
+            <origin xyz="0 0 0" rpy="0 0 0"/>
+        </xacro:inertial_sphere>
+    </link>
+    <gazebo reference="caster_wheel">
+        <material>Gazebo/White</material>
+        <mu1 value="0.001"/>
+        <mu2 value="0.001"/>
+    </gazebo>
 </robot>

Commit message: refactoring urdfs, update launchers

File: description/robot_core.xacro (robot description, xacro)
@@ -85,5 +85,5 @@
         <parent link="base_link"/>
         <child link="left_wheel"/>
-        <origin xyz="0 ${wheel_offset_y} 0" rpy="-${pi/2} 0 0" />
+        <origin xyz="${chassis_length/2 - 0.070} ${wheel_offset_y/2 + wheel_thickness/2 + 0.01} 0" rpy="-${pi/2} 0 0" />
         <axis xyz="0 0 1"/>
     </joint>
@@ -111,5 +111,5 @@
         <parent link="base_link"/>
         <child link="right_wheel"/>
-        <origin xyz="0 ${-wheel_offset_y} 0" rpy="${pi/2} 0 0" />
+        <origin xyz="${chassis_length/2 - 0.070} -${wheel_offset_y/2 + wheel_thickness/2 + 0.01} 0" rpy="${pi/2} 0 0" />
         <axis xyz="0 0 -1"/>
     </joint>
@@ -164,5 +164,5 @@
         <parent link="chassis"/>
         <child link="laser_frame"/>
-        <origin xyz="-150 0 30"/>
+        <origin xyz="${chassis_length -0.150} 0 ${chassis_height + 0.030}" rpy="0 0 0"/>
     </joint>
     <link name="laser_frame">
@@ -184,6 +184,4 @@
     <gazebo reference="laser_frame">
         <material>Gazebo/White</material>
-        <mu1 value="0.001"/>
-        <mu2 value="0.001"/>
     </gazebo>
 </robot>

Commit message: update

File: description/robot_core.xacro (robot description, xacro)
@@ -58,9 +58,9 @@
         <parent link="base_link"/>
         <child link="chassis"/>
-        <origin xyz="${-wheel_offset_x} 0 ${-wheel_offset_z}"/>
+        <origin xyz="0 0 ${-wheel_offset_z}"/>
     </joint>
     <link name="chassis">
         <visual>
-            <origin xyz="${chassis_length/2} 0 ${chassis_height/2}"/>
+            <origin xyz="0 0 0"/>
             <geometry>
                 <box size="${chassis_length} ${chassis_width} ${chassis_height}"/>
@@ -69,5 +69,5 @@
         </visual>
         <collision>
-            <origin xyz="${chassis_length/2} 0 ${chassis_height/2}"/>
+            <origin xyz="0 0 0"/>
             <geometry>
                 <box size="${chassis_length} ${chassis_width} ${chassis_height}"/>
@@ -75,5 +75,5 @@
         </collision>
         <xacro:inertial_box mass="0.5" x="${chassis_length}" y="${chassis_width}" z="${chassis_height}">
-            <origin xyz="${chassis_length/2} 0 ${chassis_height/2}" rpy="0 0 0"/>
+            <origin xyz="0 0 0" rpy="0 0 0"/>
         </xacro:inertial_box>
     </link>

Commit message: changes to geometry

File: description/robot_core.xacro (robot description, xacro)
@@ -58,5 +58,5 @@
         <parent link="base_link"/>
         <child link="chassis"/>
-        <origin xyz="-${chassis_length/2} 0 ${-wheel_offset_z}"/>
+        <origin xyz="${-chassis_length/2 + 0.070} 0 ${wheel_offset_z}"/>
     </joint>
     <link name="chassis">

Commit message: update: reversed laser_frame and changed twist_mux priority

File: description/robot_core.xacro (robot description, xacro)
@@ -161,5 +161,5 @@
     </gazebo>
     <!-- Lidar LINK -->
-    <joint name="lidar_joint" type="fixed">
+    <!-- <joint name="lidar_joint" type="fixed">
         <parent link="chassis"/>
         <child link="laser_frame"/>
@@ -181,4 +181,25 @@
             <origin xyz="0 0 0" rpy="0 0 0"/>
         </xacro:inertial_sphere>
+    </link> -->
+    <joint name="lidar_joint" type="fixed">
+        <parent link="base_link"/>
+        <child link="laser_frame"/>
+        <origin xyz="${-0.08} 0 ${chassis_height + 0.030}" rpy="0 0 ${pi}"/>
+    </joint>
+    <link name="laser_frame">
+        <visual>
+            <geometry>
+                <sphere radius="${caster_wheel_radius}"/>
+            </geometry>
+            <material name="white"/>
+        </visual>
+        <collision>
+            <geometry>
+                <sphere radius="${caster_wheel_radius}"/>
+            </geometry>
+        </collision>
+        <xacro:inertial_sphere mass="${caster_wheel_mass}" radius="${caster_wheel_radius}">
+            <origin xyz="0 0 0" rpy="0 0 0"/>
+        </xacro:inertial_sphere>
     </link>
     <gazebo reference="laser_frame">

Commit message: update: new layout for teleop with middleware

File: description/robot_core.xacro (robot description, xacro)
@@ -185,5 +185,5 @@
         <parent link="base_link"/>
         <child link="laser_frame"/>
-        <origin xyz="${-0.08} 0 ${chassis_height + 0.030}" rpy="0 0 ${pi}"/>
+        <origin xyz="${0.070-0.155} 0 ${chassis_height + 0.030}" rpy="0 0 ${pi}"/>
     </joint>
     <link name="laser_frame">

File: test.urdf (robot description, URDF)
Before this commit: robot robot, 10 links, 9 joints
Joints:
- joint lidar_joint: origin xyz=-0.08 0 0.18 rpy=0 0 3.141592653589793 -> xyz=-0.08499999999999999 0 0.18 rpy=0 0 3.141592653589793

Commit message: updated wheel joint position in relation to lidar

File: description/robot_core.xacro (robot description, xacro)
@@ -58,5 +58,5 @@
         <parent link="base_link"/>
         <child link="chassis"/>
-        <origin xyz="${-chassis_length/2 + 0.070} 0 ${wheel_offset_z}"/>
+        <origin xyz="${-chassis_length/2 + 0.075} 0 ${wheel_offset_z}"/>
     </joint>
     <link name="chassis">
@@ -85,5 +85,5 @@
         <parent link="chassis"/>
         <child link="left_wheel"/>
-        <origin xyz="${chassis_length/2 - 0.070} ${wheel_offset_y/2 + wheel_thickness/2 + 0.01} 0" rpy="-${pi/2} 0 0" />
+        <origin xyz="${chassis_length/2 - 0.075} ${wheel_offset_y/2 + wheel_thickness/2 + 0.01} 0" rpy="-${pi/2} 0 0" />
         <axis xyz="0 0 1"/>
     </joint>
@@ -111,5 +111,5 @@
         <parent link="chassis"/>
         <child link="right_wheel"/>
-        <origin xyz="${chassis_length/2 - 0.070} -${wheel_offset_y/2 + wheel_thickness/2 + 0.01} 0" rpy="${pi/2} 0 0" />
+        <origin xyz="${chassis_length/2 - 0.075} -${wheel_offset_y/2 + wheel_thickness/2 + 0.01} 0" rpy="${pi/2} 0 0" />
         <axis xyz="0 0 -1"/>
     </joint>
@@ -185,5 +185,5 @@
         <parent link="base_link"/>
         <child link="laser_frame"/>
-        <origin xyz="${0.070-0.155} 0 ${chassis_height + 0.030}" rpy="0 0 ${pi}"/>
+        <origin xyz="${0.075 - 0.15285} 0 ${chassis_height + 0.030}" rpy="0 0 ${pi}"/>
     </joint>
     <link name="laser_frame">

Commit message: update chassis height

File: description/robot_core.xacro (robot description, xacro)
@@ -58,5 +58,5 @@
         <parent link="base_link"/>
         <child link="chassis"/>
-        <origin xyz="${-chassis_length/2 + 0.075} 0 ${wheel_offset_z}"/>
+        <origin xyz="${-chassis_length/2 + 0.075} 0 ${wheel_offset_z + chassis_height}"/>
     </joint>
     <link name="chassis">

Commit message: update

File: description/robot_core.xacro (robot description, xacro)
@@ -58,5 +58,5 @@
         <parent link="base_link"/>
         <child link="chassis"/>
-        <origin xyz="${-chassis_length/2 + 0.075} 0 ${wheel_offset_z + chassis_height}"/>
+        <origin xyz="${-chassis_length/2 + 0.075} 0 ${wheel_offset_z + chassis_height/2}"/>
     </joint>
     <link name="chassis">

Commit message: update

File: description/robot_core.xacro (robot description, xacro)
@@ -58,5 +58,5 @@
         <parent link="base_link"/>
         <child link="chassis"/>
-        <origin xyz="${-chassis_length/2 + 0.075} 0 ${wheel_offset_z + chassis_height/2}"/>
+        <origin xyz="${-chassis_length/2 + 0.075} 0 ${wheel_offset_z + chassis_height}"/>
     </joint>
     <link name="chassis">

Commit message: update

File: description/robot_core.xacro (robot description, xacro)
@@ -58,5 +58,5 @@
         <parent link="base_link"/>
         <child link="chassis"/>
-        <origin xyz="${-chassis_length/2 + 0.075} 0 ${wheel_offset_z + chassis_height}"/>
+        <origin xyz="${-chassis_length/2 + 0.075} 0 ${chassis_height}"/>
     </joint>
     <link name="chassis">

Commit message: update

File: description/robot_core.xacro (robot description, xacro)
@@ -58,5 +58,5 @@
         <parent link="base_link"/>
         <child link="chassis"/>
-        <origin xyz="${-chassis_length/2 + 0.075} 0 ${chassis_height}"/>
+        <origin xyz="${-chassis_length/2 + 0.075} 0 ${wheel_radius}"/>
     </joint>
     <link name="chassis">

Commit message: update

File: description/robot_core.xacro (robot description, xacro)
@@ -4,5 +4,5 @@
     <xacro:property name="chassis_length" value="0.600"/>
     <xacro:property name="chassis_width" value="0.330"/>
-    <xacro:property name="chassis_height" value="0.150"/>
+    <xacro:property name="chassis_height" value="0.115"/>
     <xacro:property name="chassis_mass" value="15.0"/>
     <xacro:property name="wheel_radius" value="0.135"/>

Commit message: update

File: description/robot_core.xacro (robot description, xacro)
@@ -4,5 +4,5 @@
     <xacro:property name="chassis_length" value="0.600"/>
     <xacro:property name="chassis_width" value="0.330"/>
-    <xacro:property name="chassis_height" value="0.115"/>
+    <xacro:property name="chassis_height" value="0.23"/>
     <xacro:property name="chassis_mass" value="15.0"/>
     <xacro:property name="wheel_radius" value="0.135"/>

Commit message: update

File: description/robot_core.xacro (robot description, xacro)
@@ -4,5 +4,5 @@
     <xacro:property name="chassis_length" value="0.600"/>
     <xacro:property name="chassis_width" value="0.330"/>
-    <xacro:property name="chassis_height" value="0.23"/>
+    <xacro:property name="chassis_height" value="0.155"/>
     <xacro:property name="chassis_mass" value="15.0"/>
     <xacro:property name="wheel_radius" value="0.135"/>

Commit message: update

File: description/robot_core.xacro (robot description, xacro)
@@ -11,5 +11,5 @@
     <xacro:property name="wheel_offset_x" value="0.285748"/>
     <xacro:property name="wheel_offset_y" value="0.33675"/>
-    <xacro:property name="wheel_offset_z" value="0.01"/>
+    <xacro:property name="wheel_offset_z" value="-0.035"/>
     <xacro:property name="caster_wheel_radius" value="0.01"/>
     <xacro:property name="caster_wheel_mass" value="0.01"/>
@@ -58,5 +58,5 @@
         <parent link="base_link"/>
         <child link="chassis"/>
-        <origin xyz="${-chassis_length/2 + 0.075} 0 ${wheel_radius}"/>
+        <origin xyz="${-chassis_length/2 + 0.075} 0 ${wheel_radius - wheel_offset_z}"/>
     </joint>
     <link name="chassis">
@@ -85,5 +85,5 @@
         <parent link="chassis"/>
         <child link="left_wheel"/>
-        <origin xyz="${chassis_length/2 - 0.075} ${wheel_offset_y/2 + wheel_thickness/2 + 0.01} 0" rpy="-${pi/2} 0 0" />
+        <origin xyz="${chassis_length/2 - 0.075} ${wheel_offset_y/2 + wheel_thickness/2 + 0.01} wheel_offset_z" rpy="-${pi/2} 0 0" />
         <axis xyz="0 0 1"/>
     </joint>
@@ -111,5 +111,5 @@
         <parent link="chassis"/>
         <child link="right_wheel"/>
-        <origin xyz="${chassis_length/2 - 0.075} -${wheel_offset_y/2 + wheel_thickness/2 + 0.01} 0" rpy="${pi/2} 0 0" />
+        <origin xyz="${chassis_length/2 - 0.075} -${wheel_offset_y/2 + wheel_thickness/2 + 0.01} wheel_offset_z" rpy="${pi/2} 0 0" />
         <axis xyz="0 0 -1"/>
     </joint>

Commit message: update

File: description/robot_core.xacro (robot description, xacro)
@@ -85,5 +85,5 @@
         <parent link="chassis"/>
         <child link="left_wheel"/>
-        <origin xyz="${chassis_length/2 - 0.075} ${wheel_offset_y/2 + wheel_thickness/2 + 0.01} wheel_offset_z" rpy="-${pi/2} 0 0" />
+        <origin xyz="${chassis_length/2 - 0.075} ${wheel_offset_y/2 + wheel_thickness/2 + 0.01} ${wheel_offset_z}" rpy="-${pi/2} 0 0" />
         <axis xyz="0 0 1"/>
     </joint>
@@ -111,5 +111,5 @@
         <parent link="chassis"/>
         <child link="right_wheel"/>
-        <origin xyz="${chassis_length/2 - 0.075} -${wheel_offset_y/2 + wheel_thickness/2 + 0.01} wheel_offset_z" rpy="${pi/2} 0 0" />
+        <origin xyz="${chassis_length/2 - 0.075} -${wheel_offset_y/2 + wheel_thickness/2 + 0.01} ${wheel_offset_z}" rpy="${pi/2} 0 0" />
         <axis xyz="0 0 -1"/>
     </joint>

Commit message: update

File: description/robot_core.xacro (robot description, xacro)
@@ -182,8 +182,8 @@
         </xacro:inertial_sphere>
     </link> -->
-    <joint name="lidar_joint" type="fixed">
-        <parent link="base_link"/>
+    <joint name="laser_joint" type="fixed">
+        <parent link="chassis_link"/>
         <child link="laser_frame"/>
-        <origin xyz="${0.075 - 0.15285} 0 ${chassis_height + 0.030}" rpy="0 0 ${pi}"/>
+        <origin xyz="${0.075 - 0.15285} 0 ${0.030}" rpy="0 0 ${pi}"/>
     </joint>
     <link name="laser_frame">

Commit message: update

File: description/robot_core.xacro (robot description, xacro)
@@ -185,5 +185,5 @@
         <parent link="chassis_link"/>
         <child link="laser_frame"/>
-        <origin xyz="${0.075 - 0.15285} 0 ${0.030}" rpy="0 0 ${pi}"/>
+        <origin xyz="${0.075 - 0.15285} 0 0.030" rpy="0 0 ${pi}"/>
     </joint>
     <link name="laser_frame">

Commit message: update

File: description/robot_core.xacro (robot description, xacro)
@@ -183,5 +183,5 @@
     </link> -->
     <joint name="laser_joint" type="fixed">
-        <parent link="chassis_link"/>
+        <parent link="chassis"/>
         <child link="laser_frame"/>
         <origin xyz="${0.075 - 0.15285} 0 0.030" rpy="0 0 ${pi}"/>

Commit message: update

File: description/robot_core.xacro (robot description, xacro)
@@ -185,5 +185,5 @@
         <parent link="chassis"/>
         <child link="laser_frame"/>
-        <origin xyz="${0.075 - 0.15285} 0 0.030" rpy="0 0 ${pi}"/>
+        <origin xyz="${0.075 - 0.15285} 0 ${chassis_height/2 + 0.030}" rpy="0 0 ${pi}"/>
     </joint>
     <link name="laser_frame">

Commit message: update

File: description/robot_core.xacro (robot description, xacro)
@@ -185,5 +185,5 @@
         <parent link="chassis"/>
         <child link="laser_frame"/>
-        <origin xyz="${0.075 - 0.15285} 0 ${chassis_height/2 + 0.030}" rpy="0 0 ${pi}"/>
+        <origin xyz="${chassis_length/2 - 0.15285} 0 ${chassis_height/2 + 0.030}" rpy="0 0 ${pi}"/>
     </joint>
     <link name="laser_frame">

Commit message: update

File: description/robot_core.xacro (robot description, xacro)
@@ -190,5 +190,5 @@
         <visual>
             <geometry>
-                <sphere radius="${caster_wheel_radius}"/>
+                <cylinder radius="0.04" length="0.05"/>
             </geometry>
             <material name="white"/>

Commit message: update

File: description/robot_core.xacro (robot description, xacro)
@@ -192,5 +192,5 @@
                 <cylinder radius="0.04" length="0.05"/>
             </geometry>
-            <material name="white"/>
+            <material name="black"/>
         </visual>
         <collision>

Commit message: update

File: description/robot_core.xacro (robot description, xacro)
@@ -184,8 +184,8 @@
     <joint name="laser_joint" type="fixed">
         <parent link="chassis"/>
-        <child link="laser_frame"/>
+        <child link="laser"/>
         <origin xyz="${chassis_length/2 - 0.15285} 0 ${chassis_height/2 + 0.030}" rpy="0 0 ${pi}"/>
     </joint>
-    <link name="laser_frame">
+    <link name="laser">
         <visual>
             <geometry>
@@ -203,6 +203,27 @@
         </xacro:inertial_sphere>
     </link>
-    <gazebo reference="laser_frame">
+    <gazebo reference="laser">
         <material>Gazebo/White</material>
     </gazebo>
+    <joint name="imu_joint" type="fixed">
+        <parent link="chassis"/>
+        <child link="imu"/>
+        <origin xyz="${chassis_length/2 - 0.15285} 0 ${chassis_height/2 + 0.030}" rpy="0 0 ${pi}"/>
+    </joint>
+    <link name="imu">
+        <visual>
+            <geometry>
+                <cylinder radius="0.04" length="0.05"/>
+            </geometry>
+            <material name="black"/>
+        </visual>
+        <collision>
+            <geometry>
+                <sphere radius="${caster_wheel_radius}"/>
+            </geometry>
+        </collision>
+        <xacro:inertial_sphere mass="${caster_wheel_mass}" radius="${caster_wheel_radius}">
+            <origin xyz="0 0 0" rpy="0 0 0"/>
+        </xacro:inertial_sphere>
+    </link>
 </robot>

Commit message: update

File: description/robot_core.xacro (robot description, xacro)
@@ -56,5 +56,5 @@
     <!-- CHASSIS LINK -->
     <joint name="chassis_joint" type="fixed">
-        <parent link="base_link"/>
+        <parent link="base_footprint"/>
         <child link="chassis"/>
         <origin xyz="${-chassis_length/2 + 0.075} 0 ${wheel_radius - wheel_offset_z}"/>

Commit message: update

File: description/robot_core.xacro (robot description, xacro)
@@ -44,13 +44,21 @@
     </material>
     <!-- BASE LINK -->
-    <link name="base_link">
-    </link>
+    <!-- <link name="base_link">
+    </link> -->
     <!-- BASE_FOOTPRINT LINK -->
-    <joint name="base_footprint_joint" type="fixed">
+    <!-- <joint name="base_footprint_joint" type="fixed">
         <parent link="base_link"/>
         <child link="base_footprint"/>
         <origin xyz="0 0 0" rpy="0 0 0"/>
-    </joint>
+    </joint> -->
     <link name="base_footprint">
+    </link>
+    <!-- BASE LINK -->
+    <joint name="base_link_joint" type="fixed">
+        <parent link="base_footprint"/>
+        <child link="base_link"/>
+        <origin xyz="0 0 0" rpy="0 0 0"/>
+    </joint>
+    <link name="base_link">
     </link>
     <!-- CHASSIS LINK -->

Commit message: update femto

File: description/robot_core.xacro (robot description, xacro)
@@ -184,3 +184,17 @@
         <material>Gazebo/White</material>
     </gazebo>
+    <!-- femto_mega camera LINK -->
+    <!-- <joint name="femto_mega_joint" type="fixed">
+        <parent link="base_link"/>
+        <child link="femto_mega_link"/>
+        <origin xyz="0 0 0" rpy="0 0 0"/>
+    </joint>
+    <link name="femto_mega_link">
+    </link> -->
+    <xacro:femto_bolt
+            prefix="femto_mega"
+            parent="base_link"
+            use_nominal_extrinsics="true">
+        <origin xyz="0 0 0" rpy="0 0 0"/>
+    </xacro:femto_bolt>
 </robot>

Commit message: update femto location

File: description/robot_core.xacro (robot description, xacro)
@@ -185,12 +185,4 @@
     </gazebo>
     <!-- femto_mega camera LINK -->
-    <!-- <joint name="femto_mega_joint" type="fixed">
-        <parent link="base_link"/>
-        <child link="femto_mega_link"/>
-        <origin xyz="0 0 0" rpy="0 0 0"/>
-    </joint>
-    <link name="femto_mega_link">
-    </link> -->
-     <!-- femto_bolt xacro file -->
     <xacro:include filename="femto_mega.urdf.xacro" />
     <xacro:femto_bolt
@@ -198,5 +190,36 @@
             parent="base_link"
             use_nominal_extrinsics="true">
-        <origin xyz="0 0 0" rpy="0 0 0"/>
+        <origin xyz=".1 0 1.35" rpy="0 .5 0"/>
     </xacro:femto_bolt>
+    <!-- Beam joint connecting base_link to beam -->
+<joint name="femto_mega_beam_joint" type="fixed">
+  <parent link="base_link"/>
+  <child link="femto_mega_beam_link"/>
+  <!-- Adjust this to match the midpoint between base_link and femto_mega_base_link -->
+  <origin xyz="0.05 0 0.675" rpy="0 0 0"/>
+</joint>
+<!-- Beam link -->
+<link name="femto_mega_beam_link">
+  <visual>
+    <!-- Adjust size and placement to match the camera mount -->
+    <origin xyz="0 0 0.2" rpy="0 0 0"/>
+    <geometry>
+      <box size="0.05 0.05 1.1"/> <!-- (x, y, z) length of the beam -->
+    </geometry>
+    <material name="beam_grey">
+      <color rgba="0.5 0.5 0.5 1.0"/>
+    </material>
+  </visual>
+  <collision>
+    <origin xyz="0 0 0" rpy="0 0 0"/>
+    <geometry>
+      <box size="0.1 0.02 1.35"/>
+    </geometry>
+  </collision>
+  <inertial>
+    <mass value="0.1"/>
+    <origin xyz="0 0 0" rpy="0 0 0"/>
+    <inertia ixx="0.01" ixy="0" ixz="0" iyy="0.01" iyz="0" izz="0.01"/>
+  </inertial>
+</link>
 </robot>

Commit message: update urdf

File: description/robot_core.xacro (robot description, xacro)
@@ -190,5 +190,5 @@
             parent="base_link"
             use_nominal_extrinsics="true">
-        <origin xyz=".1 0 1.35" rpy="0 .5 0"/>
+        <origin xyz=".07 0 1.00" rpy="0 .5 0"/>
     </xacro:femto_bolt>
     <!-- Beam joint connecting base_link to beam -->
